File: ATtiny10_Writer.sch (EAGLE design)
At the start: 5 parts, among them CON1 AVR_ISP, J1 SOT23-6_2_SOCKET

Commit message: complete all
Parts:
- added H1, H2, H3, H4: MOUNT-HOLE3.2, holes:MOUNT-HOLE3.2
- added J2: ZX62-B-5PA(33), ZX62-B-5PA_33_:ZX62-B-5PA(33)
- added LED2: (no value), led:LEDCHIP-LED0603
- added R2: (no value), rcl:R-EU_R0603
Connections:
- new net N$2: LED2.C, R2.2
- net GND: now also J2.5, J2.SHIELD, R2.1
- net VCC: now also J2.1, LED2.A
Changed lines of the file:
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@@
 <?xml version="1.0" encoding="utf-8"?>
 <!DOCTYPE eagle SYSTEM "eagle.dtd">
-<eagle version="9.4.2">
+<eagle version="9.1.3">
 <drawing>
 <settings>
@@
 <part name="R1" library="rcl" library_urn="urn:adsk.eagle:library:334" deviceset="R-EU_" device="R0603" package3d_urn="urn:adsk.eagle:package:23555/3"/>
 <part name="LED1" library="led" library_urn="urn:adsk.eagle:library:259" deviceset="LED" device="CHIP-LED0603" package3d_urn="urn:adsk.eagle:package:15819/3"/>
+<part name="J2" library="ZX62-B-5PA_33_" deviceset="ZX62-B-5PA(33)" device=""/>
+<part name="H1" library="holes" library_urn="urn:adsk.eagle:library:237" deviceset="MOUNT-HOLE" device="3.2" package3d_urn="urn:adsk.eagle:package:14275/1"/>
+<part name="H2" library="holes" library_urn="urn:adsk.eagle:library:237" deviceset="MOUNT-HOLE" device="3.2" package3d_urn="urn:adsk.eagle:package:14275/1"/>
+<part name="H3" library="holes" library_urn="urn:adsk.eagle:library:237" deviceset="MOUNT-HOLE" device="3.2" package3d_urn="urn:adsk.eagle:package:14275/1"/>
+<part name="H4" library="holes" library_urn="urn:adsk.eagle:library:237" deviceset="MOUNT-HOLE" device="3.2" package3d_urn="urn:adsk.eagle:package:14275/1"/>
+<part name="P+5" library="supply1" library_urn="urn:adsk.eagle:library:371" deviceset="VCC" device=""/>
+<part name="SUPPLY6" library="supply2" library_urn="urn:adsk.eagle:library:372" deviceset="GND" device=""/>
+<part name="SUPPLY7" library="supply2" library_urn="urn:adsk.eagle:library:372" deviceset="GND" device=""/>
+<part name="R2" library="rcl" library_urn="urn:adsk.eagle:library:334" deviceset="R-EU_" device="R0603" package3d_urn="urn:adsk.eagle:package:23555/3"/>
+<part name="LED2" library="led" library_urn="urn:adsk.eagle:library:259" deviceset="LED" device="CHIP-LED0603" package3d_urn="urn:adsk.eagle:package:15819/3"/>
+<part name="P+6" library="supply1" library_urn="urn:adsk.eagle:library:371" deviceset="VCC" device=""/>
 </parts>
 <sheets>
@@
 <attribute name="VALUE" x="112.395" y="15.748" size="1.778" layer="96" rot="R90"/>
 </instance>
+<instance part="J2" gate="G$1" x="139.7" y="12.7"/>
+<instance part="H1" gate="G$1" x="116.84" y="63.5"/>
+<instance part="H2" gate="G$1" x="142.24" y="63.5"/>
+<instance part="H3" gate="G$1" x="116.84" y="55.88"/>
+<instance part="H4" gate="G$1" x="142.24" y="55.88"/>
+<instance part="P+5" gate="VCC" x="129.54" y="27.94" smashed="yes">
+<attribute name="VALUE" x="127" y="25.4" size="1.778" layer="96" rot="R90"/>
+</instance>
+<instance part="SUPPLY6" gate="GND" x="129.54" y="-2.54" smashed="yes">
+<attribute name="VALUE" x="127.635" y="-5.715" size="1.778" layer="96"/>
+</instance>
+<instance part="SUPPLY7" gate="GND" x="116.84" y="2.54" smashed="yes">
+<attribute name="VALUE" x="114.935" y="-0.635" size="1.778" layer="96"/>
+</instance>
+<instance part="R2" gate="G$1" x="116.84" y="10.16" smashed="yes" rot="R90">
+<attribute name="NAME" x="115.3414" y="6.35" size="1.778" layer="95" rot="R90"/>
+<attribute name="VALUE" x="120.142" y="6.35" size="1.778" layer="96" rot="R90"/>
+</instance>
+<instance part="LED2" gate="G$1" x="116.84" y="20.32" smashed="yes">
+<attribute name="NAME" x="120.396" y="15.748" size="1.778" layer="95" rot="R90"/>
+<attribute name="VALUE" x="122.555" y="15.748" size="1.778" layer="96" rot="R90"/>
+</instance>
+<instance part="P+6" gate="VCC" x="116.84" y="27.94" smashed="yes">
+<attribute name="VALUE" x="114.3" y="25.4" size="1.778" layer="96" rot="R90"/>
+</instance>
 </instances>
 <busses>
@@
 <pinref part="R1" gate="G$1" pin="1"/>
 </segment>
+<segment>
+<pinref part="J2" gate="G$1" pin="5"/>
+<pinref part="J2" gate="G$1" pin="SHIELD"/>
+<wire x1="129.54" y1="10.16" x2="129.54" y2="5.08" width="0.1524" layer="91"/>
+<wire x1="129.54" y1="5.08" x2="129.54" y2="0" width="0.1524" layer="91"/>
+<junction x="129.54" y="5.08"/>
+<pinref part="SUPPLY6" gate="GND" pin="GND"/>
+</segment>
+<segment>
+<pinref part="SUPPLY7" gate="GND" pin="GND"/>
+<pinref part="R2" gate="G$1" pin="1"/>
+</segment>
 </net>
 <net name="VCC" class="0">
@@
 <wire x1="91.44" y1="17.78" x2="91.44" y2="12.7" width="0.1524" layer="91"/>
 </segment>
+<segment>
+<pinref part="P+5" gate="VCC" pin="VCC"/>
+<pinref part="J2" gate="G$1" pin="1"/>
+<wire x1="129.54" y1="25.4" x2="129.54" y2="20.32" width="0.1524" layer="91"/>
+</segment>
+<segment>
+<pinref part="P+6" gate="VCC" pin="VCC"/>
+<pinref part="LED2" gate="G$1" pin="A"/>
+<wire x1="116.84" y1="25.4" x2="116.84" y2="22.86" width="0.1524" layer="91"/>
+</segment>
 </net>
 <net name="N$1" class="0">
@@
 </segment>
 </net>
+<net name="N$2" class="0">
+<segment>
+<pinref part="R2" gate="G$1" pin="2"/>
+<pinref part="LED2" gate="G$1" pin="C"/>
+</segment>
+</net>
